Commit message: Update world xy joint limits.

File: models/iiwa/mobile_iiwa.urdf (robot description, URDF)
Before this commit: robot mobile_iiwa, 14 links, 13 joints
Joints:
- joint world_x_joint: limit lower=-2.0 upper=2.0 effort=1000 velocity=0.5 -> lower=-1.0 upper=5.0 effort=1000 velocity=0.5
- joint world_y_joint: limit lower=-2.0 upper=2.0 effort=1000 velocity=0.5 -> lower=-1.0 upper=5.0 effort=1000 velocity=0.5

Commit message: Make world theta continuous revolute.

File: models/iiwa/mobile_iiwa.urdf (robot description, URDF)
Before this commit: robot mobile_iiwa, 14 links, 13 joints
Joints:
- joint iiwa_base_theta_joint: limit lower=-3.1416 upper=3.1416 effort=1000 velocity=3.1416 -> effort=1000 velocity=3.1416; type revolute -> continuous

Commit message: Take away the continuous revolute base joint, so the iiwa doesn't spin around a bunch.

File: models/iiwa/mobile_iiwa.urdf (robot description, URDF)
Before this commit: robot mobile_iiwa, 14 links, 13 joints
Joints:
- joint iiwa_base_theta_joint: limit effort=1000 velocity=3.1416 -> lower=-3.1416 upper=3.1416 effort=1000 velocity=3.1416; type continuous -> revolute

Commit message: Add transmission to mobile_iiwa.urdf, so it can be used with InverseDynamicsDriver.

File: models/iiwa/mobile_iiwa.urdf (robot description, URDF)
Before this commit: robot mobile_iiwa, 14 links, 13 joints
Joints:
- removed joint world_x_joint
- removed joint world_y_joint
- added joint base_x_joint: type prismatic, parent base, child iiwa_base_x, origin xyz=0 0 0 rpy=0 0 0, axis 1 0 0, limit lower=-1.0 upper=5.0 effort=1000 velocity=0.5
- added joint base_y_joint: type prismatic, parent iiwa_base_x, child iiwa_base_y, origin xyz=0 0 0 rpy=0 0 0, axis 0 1 0, limit lower=-1.0 upper=5.0 effort=1000 velocity=0.5

Commit message: Add visual and collision geometry associated to the lift joint.

File: models/iiwa/mobile_iiwa.urdf (robot description, URDF)
Before this commit: robot mobile_iiwa, 14 links, 13 joints
Links:
- added link iiwa_base_z_column; collision box size=0.3 0.3 1.0; visual box size=0.3 0.3 1.0
Joints:
- added joint iiwa_base_z_column_joint: type fixed, parent iiwa_base_theta, child iiwa_base_z_column, origin xyz=0 0 -0.5 rpy=0 0 0

Commit message: Fix where the lift joint geometry is attached.

File: models/iiwa/mobile_iiwa.urdf (robot description, URDF)
Before this commit: robot mobile_iiwa, 15 links, 14 joints
Joints:
- joint iiwa_base_z_column_joint: parent iiwa_base_theta -> iiwa_link_0

Commit message: Make the robot taller to reach high shelves.

File: models/iiwa/mobile_iiwa.urdf (robot description, URDF)
Before this commit: robot mobile_iiwa, 15 links, 14 joints
Links:
- link iiwa_base_z_column: geometry collision box size=0.3 0.3 2.0; visual box size=0.3 0.3 2.0
Joints:
- joint iiwa_base_z_column_joint: origin xyz=0 0 -0.5 rpy=0 0 0 -> xyz=0 0 -1.0 rpy=0 0 0
- joint iiwa_base_z_joint: limit lower=0.0 upper=1.0 effort=1000 velocity=0.5 -> lower=0.0 upper=2.0 effort=1000 velocity=0.5

Commit message: Remove xy prismaticjoint limits.

File: models/iiwa/mobile_iiwa.urdf (robot description, URDF)
Before this commit: robot mobile_iiwa, 15 links, 14 joints
Joints:
- joint base_x_joint: limit lower=-1.0 upper=5.0 effort=1000 velocity=0.5 -> effort=1000 velocity=0.5
- joint base_y_joint: limit lower=-1.0 upper=5.0 effort=1000 velocity=0.5 -> effort=1000 velocity=0.5
