Commit message: Replace Zerith base collision hull with box proxies
Add filtered initial-penetration reporting for contact diagnostics.

File: models/zerith_drake/urdf/zerith_drake.urdf (robot description, URDF)
Before this commit: robot ZR_H1PRO-1.2.00.H.V4.3_URDF_2025.12.02, 35 links, 34 joints
Links:
- link dipan_link: geometry collision box size=0.188 0.196 0.035; collision box size=0.235 0.23 1.1

Commit message: Replace Zerith wrist and gripper collision hulls

File: models/zerith_drake/urdf/zerith_drake.urdf (robot description, URDF)
Before this commit: robot ZR_H1PRO-1.2.00.H.V4.3_URDF_2025.12.02, 35 links, 34 joints
Links:
- link left_end_effector_link: geometry collision box size=0.0015 0.029 0.008; collision box size=0.0015 0.029 0.008
- link left_jaw_left_finger_link: geometry collision box size=0.018 0.027 0.055; collision box size=0.025 0.013 0.035
- link left_jaw_right_finger_link: geometry collision box size=0.018 0.027 0.055; collision box size=0.025 0.013 0.035
- link left_wrist_pitch_link: geometry collision box size=0.018 0.145 0.04; collision box size=0.034 0.06 0.05
- link left_wrist_roll_link: geometry collision cylinder length=0.096 radius=0.031; visual mesh filename=package://zerith_drake/meshes/left_wrist_roll_link.obj
- link left_wrist_yaw_link: geometry collision cylinder length=0.065 radius=0.025; visual mesh filename=package://zerith_drake/meshes/left_wrist_yaw_link.obj
- link right_end_effector_link: geometry collision box size=0.0015 0.029 0.008; collision box size=0.0015 0.029 0.008
- link right_jaw_left_finger_link: geometry collision box size=0.018 0.027 0.055; collision box size=0.025 0.013 0.035
- link right_jaw_right_finger_link: geometry collision box size=0.018 0.027 0.055; collision box size=0.025 0.013 0.035
- link right_wrist_pitch_link: geometry collision box size=0.018 0.145 0.04; collision box size=0.034 0.06 0.05
- link right_wrist_roll_link: geometry collision cylinder length=0.096 radius=0.031; visual mesh filename=package://zerith_drake/meshes/right_wrist_roll_link.obj
- link right_wrist_yaw_link: geometry collision cylinder length=0.065 radius=0.025; visual mesh filename=package://zerith_drake/meshes/right_wrist_yaw_link.obj

Commit message: Fix Zerith finger contact geometry and calibrate gripper opening

File: models/zerith_drake/urdf/zerith_drake.urdf (robot description, URDF)
Before this commit: robot ZR_H1PRO-1.2.00.H.V4.3_URDF_2025.12.02, 35 links, 34 joints
Links:
- link left_jaw_left_finger_link: geometry collision box size=0.018 0.027 0.055; collision mesh filename=package://zerith_drake/meshes/left_jaw_left_finger_link_mid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
- link left_jaw_right_finger_link: geometry collision box size=0.018 0.027 0.055; collision mesh filename=package://zerith_drake/meshes/left_jaw_right_finger_link_mi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
- link right_jaw_left_finger_link: geometry collision box size=0.018 0.027 0.055; collision mesh filename=package://zerith_drake/meshes/right_jaw_left_finger_link_mi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
- link right_jaw_right_finger_link: geometry collision box size=0.018 0.027 0.055; collision mesh filename=package://zerith_drake/meshes/right_jaw_right_finger_link_m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
Joints:
- joint left_jaw_left_finger_joint: limit lower=-0.04 upper=0 effort=120 velocity=0.25 -> lower=-0.03814 upper=0 effort=120 velocity=0.25
- joint left_jaw_right_finger_joint: limit lower=0 upper=0.04 effort=120 velocity=0.25 -> lower=0 upper=0.03814 effort=120 velocity=0.25
- joint right_jaw_left_finger_joint: limit lower=-0.04 upper=0 effort=120 velocity=0.25 -> lower=-0.03814 upper=0 effort=120 velocity=0.25
- joint right_jaw_right_finger_joint: limit lower=0 upper=0.04 effort=120 velocity=0.25 -> lower=0 upper=0.03814 effort=120 velocity=0.25
